File: PRACTICA03/LAVIGNA_GONZALO/osc.sch (KiCad schematic (older format))
At the start: 8 parts, among them J201 Conn_01x02, U201 40106

Commit message: Agregado de liberias, exportacion proyecto a Altium Tratando de encontrar Aduino Mega Shield para Kicad con nombres parecidos capaz convenga usarla.
Parts:
- added U202: XC6SLX9-2TQG144C, SPARTAN6:TQ144, symbol XC6SLX9-2TQG144C:XC6SLX9-2TQG144C
Changed lines of the file:
@@
 Wire Wire Line
 	2700 2150 2550 2150
+$Comp
+L XC6SLX9-2TQG144C:XC6SLX9-2TQG144C U202
+U 1 1 5BB8A4C7
+P 13850 2300
+F 0 "U202" H 13850 2300 50  0001 L BNN
+F 1 "XC6SLX9-2TQG144C" H 13850 2300 50  0001 L BNN
+F 2 "SPARTAN6:TQ144" H 13850 2300 50  0001 L BNN
+F 3 "TQFP-144 Xilinx" H 13850 2300 50  0001 L BNN
+F 4 "FPGA SpartanÂ®-6 LX Family 9152 Cells 45nm _CMOS_ Technology 1.2V 144-Pin TQFP" H 13850 2300 50  0001 L BNN "Campo4"
+F 5 "XC6SLX9-2TQG144C" H 13850 2300 50  0001 L BNN "Campo5"
+F 6 "None" H 13850 2300 50  0001 L BNN "Campo6"
+F 7 "Xilinx" H 13850 2300 50  0001 L BNN "Campo7"
+F 8 "Unavailable" H 13850 2300 50  0001 L BNN "Campo8"
+	1    13850 2300
+	1    0    0    -1
+$EndComp
 $EndSCHEMATC
