File: PRACTICA_FINAL/PROJECTO_KICAD/FINAL/FPGA-CORE.sch (KiCad schematic (older format))
At the start: 7 parts

Commit message: Actualizado el esquematico de la FPGA, terminada todas las conexiones quedan los pines jerarquicos nada mas a nivel esquematico.
Parts:
- added R? (x14): 390, symbol Papilio_DUO-eagle-import:R-NORMAL0603
- added R?: 47K, symbol Papilio_DUO-eagle-import:R-NORMAL0805
- added R?: 4.7K, symbol Papilio_DUO-eagle-import:R-NORMAL0603
- added U?: EVQQ2, symbol Papilio_DUO-eagle-import:EVQQ2
Connections:
- net labels added: +5V, AD0-JTAG_TCK, AD1-JTAG_TDI, AD2-JTAG_TDO, AD3-JTAG_TMS, AD4-DTR, ARD_RESET, AREF, ATMEGA_A0, ATMEGA_A1, BD0_TXD/MPSSE_TCK, BD1_RXD/MPSSE_TDI, BD2_MPSSE_TDO, BD3_MPSSE_TMS, BD4-DTR, FLASH_CS, FLASH_SCK, FLASH_SI, FLASH_SO, GND, MEGA_D0, MEGA_D1, MEGA_D10, MEGA_D11, MEGA_D12, MEGA_D13, MEGA_D14, MEGA_D15, MEGA_D16, MEGA_D17, MEGA_D18, MEGA_D19, MEGA_D2, MEGA_D20, MEGA_D21, MEGA_D22, MEGA_D23, MEGA_D24, MEGA_D25, MEGA_D26, MEGA_D27, MEGA_D28/A5, MEGA_D29, MEGA_D3, MEGA_D30/A4, MEGA_D31, MEGA_D32/A3, MEGA_D33, MEGA_D34/A2, MEGA_D35, MEGA_D36, MEGA_D37, MEGA_D38, MEGA_D39, MEGA_D4, MEGA_D40, MEGA_D41, MEGA_D42, MEGA_D43, MEGA_D44, MEGA_D45, MEGA_D46, MEGA_D47, MEGA_D48, MEGA_D49, MEGA_D5, MEGA_D50, MEGA_D51, MEGA_D52, MEGA_D53, MEGA_D6, MEGA_D7, MEGA_D8, MEGA_D9, MEGA_SHIELD_BUS, OSC_IN, SRAM_A0, SRAM_A1, SRAM_A10, SRAM_A11, SRAM_A12, SRAM_A13, SRAM_A14, SRAM_A15, SRAM_A16, SRAM_A17, SRAM_A18, SRAM_A19, SRAM_A2, SRAM_A20, SRAM_A3, SRAM_A4, SRAM_A5, SRAM_A6, SRAM_A7, SRAM_A8, SRAM_A9, SRAM_BUS, SRAM_D0, SRAM_D1, SRAM_D2, SRAM_D3, SRAM_D4, SRAM_D5, SRAM_D6, SRAM_D7, SW1, ~SRAM_CS, ~SRAM_OE, ~SRAM_WE
- wire segments 13 -> 300
- no-connect marks 0 -> 1
Other:
- note added: "RESET"

Commit message: Actualizado el esquematico se enumera igual que el pdf. Se asignan todas las huellas lo unico que falta es la huella de un Arduino superpuesto Se corre DRC de esquematico y tambien se pasa a .NET y se levanta en el Kicad PCB sin errores
Parts:
- R10, R11, R12, R13, R14, R15, R16, R17, R18, R19, R20, R21, R32, R8, R9: renamed from R?; footprint (none) -> Papilio_DUO:0603
- R31: renamed from R?; footprint (none) -> Papilio_DUO:0805
- S1: renamed from U?; footprint (none) -> Papilio_DUO:TQ144
- SRAM1: renamed from U?; footprint (none) -> Papilio_DUO:TSOP44-II
- SW2: renamed from U?; footprint (none) -> Papilio_DUO:EVQ-Q2
- U1: renamed from U?; footprint (none) -> Papilio_DUO:ARDUINO_MEGA_SHIELD
Connections:
- wire segments 300 -> 297
- no-connect marks 1 -> 3
Other:
- note added: "ATMEGA"
- note added: "JTAG FTDI"
- note added: "JTAG XILINX"
- note added: "MEMORIA PROGRAMACION"
- note added: "RESET MANUAL Y CLOCK"
