File: PRACTICA_FINAL/PROJECTO_KICAD/FINAL/FPGA-POWER.sch (KiCad schematic (older format))
At the start: 27 parts

Commit message: Actualizado el esquematico se enumera igual que el pdf. Se asignan todas las huellas lo unico que falta es la huella de un Arduino superpuesto Se corre DRC de esquematico y tambien se pasa a .NET y se levanta en el Kicad PCB sin errores
Parts:
- C10, C11, C13, C21, C22, C23, C24, C25, C26, C32, C33, C35, C36, C4, C5, C6, C7: renamed from C?; footprint (none) -> Papilio_DUO:0603
- C12: renamed from C?; footprint (none) -> Papilio_DUO:0805
- S1: renamed from U?; footprint (none) -> Papilio_DUO:TQ144
- WING_POWER1, WING_POWER2, WING_POWER3, WING_POWER4, WING_POWER5, WING_POWER6: renamed from WING_POWER?; footprint (none) -> Papilio_DUO:POWER_NO_TEXT
Connections:
- no-connect marks 0 -> 6
