File: PRACTICA_FINAL/PROJECTO_KICAD/FINAL/Power.sch (KiCad schematic (older format))
At the start: 14 parts

Commit message: Actualizado el esquematico se enumera igual que el pdf. Se asignan todas las huellas lo unico que falta es la huella de un Arduino superpuesto Se corre DRC de esquematico y tambien se pasa a .NET y se levanta en el Kicad PCB sin errores
Parts:
- C1, C2, C3: renamed from C?; footprint (none) -> Papilio_DUO:0805
- L1, L2: renamed from L?; footprint (none) -> Papilio_DUO:VLS3015
- PWR1: value GREEN -> Green; footprint (none) -> Papilio_DUO:CHIP-LED0805
- PWRIN1: renamed from JP?; footprint (none) -> Papilio_DUO:JP1
- PWRSEL1: renamed from JP?; value PWRSEL1 -> JP2E; footprint (none) -> Papilio_DUO:JP2
- R2, R3, R4, R5, R6: renamed from R?; footprint (none) -> Papilio_DUO:0603
- U2: renamed from U?; footprint (none) -> Papilio_DUO:MSOP10
Connections:
- wire segments 45 -> 50
