File: PRACTICA_FINAL/PROJECTO_KICAD/FINAL/Arduino.sch (KiCad schematic (older format))
At the start: 16 parts

Commit message: Terminada la hoja del FTDI y POWER y Arduino.bak FPGA terminado Power y Pheripheral. Lo principal de la cuestion del bnloque FPGA estan puestos los componentyes. Queda revisar globales y pasarlas a locales despues de eso. Un proyecto con muchas cosas globales se hace muy dificil de seguir.
Parts:
- added C?: 1uF, symbol Papilio_DUO-eagle-import:C0603
Connections:
- net labels added: 5V_ARDUINO, AREF, ATMEGA_A0, ATMEGA_A1, ATMEGA_D0/RX, ATMEGA_D1/TX, ATMEGA_D2, ATMEGA_D3, ATMEGA_D4, ATMEGA_D5*, ATMEGA_D6*, ATMEGA_D7, ATMEGA_IO10*, ATMEGA_IO11*, ATMEGA_IO12, ATMEGA_IO13*, ATMEGA_IO8, ATMEGA_IO9*, MEGA_D14, MEGA_D15, MEGA_D16, MEGA_D28/A5, MEGA_D30/A4, MEGA_D32/A3, MEGA_D34/A2, NC
- net labels removed: ATMETA_IO13*, UGND
- wire segments 95 -> 135

Commit message: Actualizado el esquematico se enumera igual que el pdf. Se asignan todas las huellas lo unico que falta es la huella de un Arduino superpuesto Se corre DRC de esquematico y tambien se pasa a .NET y se levanta en el Kicad PCB sin errores
Parts:
- AVRUSB1: renamed from J?; footprint (none) -> Papilio_DUO:CON2_USB_MICRO_B_AT
- C101, C103, C104, C105, C106, C107: renamed from C?; footprint (none) -> Papilio_DUO:0603
- C102: renamed from C?; value C0603 -> 100nF; footprint (none) -> Papilio_DUO:0603
- L100: renamed from L?; footprint (none) -> Papilio_DUO:0805
- LED1: renamed from LED?; value YELLOW -> Yellow; footprint (none) -> Papilio_DUO:CHIP-LED0805
- R1, R22: renamed from R?; footprint (none) -> Papilio_DUO:0805
- R109, R7: renamed from R?; footprint (none) -> Papilio_DUO:0603
- R110: renamed from R?; value 4.7K -> 10K; footprint (none) -> Papilio_DUO:0603
- U101: renamed from U?; footprint (none) -> Papilio_DUO:QFN44ML7X7
- Y1: renamed from Y?; footprint (none) -> Papilio_DUO:CRYSTAL-3.2-2.5
Connections:
- wire segments 135 -> 137
- no-connect marks 0 -> 16
Changed lines of the file:
@@
 $Descr A4 11693 8268
 encoding utf-8
-Sheet 8 8
+Sheet 7 8
 Title ""
 Date ""
@@
 $EndDescr
 $Comp
-L Papilio_DUO-eagle-import:MYCON2_USB-MINI-B J?
+L Papilio_DUO-eagle-import:MYCON2_USB-MINI-B AVRUSB1
 U 1 1 5BB94B08
 P 4450 5500
-F 0 "J?" H 4450 5986 59  0000 C CNN
+F 0 "AVRUSB1" H 4450 5986 59  0000 C CNN
 F 1 "MYCON2_USB-MINI-B" H 4450 5881 59  0000 C CNN
-F 2 "" H 4450 5500 50  0001 C CNN
+F 2 "Papilio_DUO:CON2_USB_MICRO_B_AT" H 4450 5500 50  0001 C CNN
 F 3 "" H 4450 5500 50  0001 C CNN
 	1    4450 5500
@@
 $EndComp
 $Comp
-L Papilio_DUO-eagle-import:R-NORMAL0603 R?
+L Papilio_DUO-eagle-import:R-NORMAL0603 R1
 U 1 1 5BB94C94
 P 6050 5250
-F 0 "R?" H 6050 5050 50  0000 C CNN
+F 0 "R1" H 6050 5050 50  0000 C CNN
 F 1 "22R" H 6050 5141 50  0000 C CNN
-F 2 "" V 5980 5250 50  0001 C CNN
+F 2 "Papilio_DUO:0805" V 5980 5250 50  0001 C CNN
 F 3 "~" H 6050 5250 50  0001 C CNN
 	1    6050 5250
@@
 $EndComp
 $Comp
-L Papilio_DUO-eagle-import:R-NORMAL0603 R?
+L Papilio_DUO-eagle-import:R-NORMAL0603 R7
 U 1 1 5BB94E64
 P 8050 4950
-F 0 "R?" V 8096 4887 50  0000 R CNN
+F 0 "R7" V 8096 4887 50  0000 R CNN
 F 1 "4.7K" V 8005 4887 50  0000 R CNN
-F 2 "" V 7980 4950 50  0001 C CNN
+F 2 "Papilio_DUO:0603" V 7980 4950 50  0001 C CNN
 F 3 "~" H 8050 4950 50  0001 C CNN
 	1    8050 4950
@@
 $EndComp
 $Comp
-L Papilio_DUO-eagle-import:R-NORMAL0603 R?
+L Papilio_DUO-eagle-import:R-NORMAL0603 R22
 U 1 1 5BB95551
 P 6050 5650
-F 0 "R?" H 6050 5450 50  0000 C CNN
+F 0 "R22" H 6050 5450 50  0000 C CNN
 F 1 "22R" H 6050 5541 50  0000 C CNN
-F 2 "" V 5980 5650 50  0001 C CNN
+F 2 "Papilio_DUO:0805" V 5980 5650 50  0001 C CNN
 F 3 "~" H 6050 5650 50  0001 C CNN
 	1    6050 5650
@@
 $EndComp
 $Comp
-L Papilio_DUO-eagle-import:LEDCHIP-LED0805 LED?
+L Papilio_DUO-eagle-import:LEDCHIP-LED0805 LED1
 U 1 1 5BB957E2
 P 8050 5400
-F 0 "LED?" H 8128 5403 59  0000 L CNN
-F 1 "YELLOW" H 8128 5298 59  0000 L CNN
-F 2 "" H 8050 5400 50  0001 C CNN
+F 0 "LED1" H 8128 5403 59  0000 L CNN
+F 1 "Yellow" H 8128 5298 59  0000 L CNN
+F 2 "Papilio_DUO:CHIP-LED0805" H 8050 5400 50  0001 C CNN
 F 3 "" H 8050 5400 50  0001 C CNN
 	1    8050 5400
@@
 	4850 1000 5400 1000
 $Comp
-L Papilio_DUO-eagle-import:C0603 C?
+L Papilio_DUO-eagle-import:C0603 C105
 U 1 1 5BB987E9
 P 4500 950
-F 0 "C?" V 4540 862 42  0000 R CNN
+F 0 "C105" V 4540 862 42  0000 R CNN
 F 1 "100nF" V 4461 862 42  0000 R CNN
-F 2 "" H 4500 950 50  0001 C CNN
+F 2 "Papilio_DUO:0603" H 4500 950 50  0001 C CNN
 F 3 "" H 4500 950 50  0001 C CNN
 	1    4500 950
@@
 $EndComp
 $Comp
-L Papilio_DUO-eagle-import:C0603 C?
+L Papilio_DUO-eagle-import:C0603 C101
 U 1 1 5BB98903
 P 4100 950
-F 0 "C?" V 4140 1038 42  0000 L CNN
+F 0 "C101" V 4140 1038 42  0000 L CNN
 F 1 "100nF" V 4061 1038 42  0000 L CNN
-F 2 "" H 4100 950 50  0001 C CNN
+F 2 "Papilio_DUO:0603" H 4100 950 50  0001 C CNN
 F 3 "" H 4100 950 50  0001 C CNN
 	1    4100 950
@@
 	5400 1700 3200 1700
 $Comp
-L Papilio_DUO-eagle-import:R-NORMAL0603 R?
+L Papilio_DUO-eagle-import:R-NORMAL0603 R109
 U 1 1 5BBA6335
 P 2900 1600
-F 0 "R?" V 2946 1537 50  0000 R CNN
+F 0 "R109" V 2946 1537 50  0000 R CNN
 F 1 "1M" V 2855 1537 50  0000 R CNN
-F 2 "" H 2900 1600 50  0001 C CNN
+F 2 "Papilio_DUO:0603" H 2900 1600 50  0001 C CNN
 F 3 "" H 2900 1600 50  0001 C CNN
 	1    2900 1600
@@
 XTAL1
 $Comp
-L Papilio_DUO-eagle-import:CRYSTAL-3.2-2.5 Y?
+L Papilio_DUO-eagle-import:CRYSTAL-3.2-2.5 Y1
 U 1 1 5BBACA7A
 P 2350 1600
-F 0 "Y?" V 2450 1500 59  0000 R CNN
+F 0 "Y1" V 2450 1500 59  0000 R CNN
 F 1 "16Mhz KX-7" V 2200 1550 59  0000 R CNN
-F 2 "" H 2350 1600 50  0001 C CNN
+F 2 "Papilio_DUO:CRYSTAL-3.2-2.5" H 2350 1600 50  0001 C CNN
 F 3 "" H 2350 1600 50  0001 C CNN
 	1    2350 1600
@@
 $EndComp
 $Comp
-L Papilio_DUO-eagle-import:C0603 C?
+L Papilio_DUO-eagle-import:C0603 C106
 U 1 1 5BBAF979
 P 1700 1400
-F 0 "C?" H 1700 1607 42  0000 C CNN
+F 0 "C106" H 1700 1607 42  0000 C CNN
 F 1 "22pF" H 1700 1528 42  0000 C CNN
-F 2 "" H 1700 1400 50  0001 C CNN
+F 2 "Papilio_DUO:0603" H 1700 1400 50  0001 C CNN
 F 3 "" H 1700 1400 50  0001 C CNN
 	1    1700 1400
@@
 $EndComp
 $Comp
-L Papilio_DUO-eagle-import:C0603 C?
+L Papilio_DUO-eagle-import:C0603 C107
 U 1 1 5BBAF9D9
 P 1700 1800
-F 0 "C?" H 1700 1700 42  0000 C CNN
+F 0 "C107" H 1700 1700 42  0000 C CNN
 F 1 "22pF" H 1700 1600 42  0000 C CNN
-F 2 "" H 1700 1800 50  0001 C CNN
+F 2 "Papilio_DUO:0603" H 1700 1800 50  0001 C CNN
 F 3 "" H 1700 1800 50  0001 C CNN
 	1    1700 1800
@@
 	1350 2100 1350 1800
 $Comp
-L Papilio_DUO-eagle-import:R-NORMAL0603 R?
+L Papilio_DUO-eagle-import:R-NORMAL0603 R110
 U 1 1 5BBBA97E
 P 9650 1150
-F 0 "R?" V 9696 1087 50  0000 R CNN
-F 1 "4.7K" V 9605 1087 50  0000 R CNN
-F 2 "" V 9580 1150 50  0001 C CNN
+F 0 "R110" V 9696 1087 50  0000 R CNN
+F 1 "10K" V 9605 1087 50  0000 R CNN
+F 2 "Papilio_DUO:0603" V 9580 1150 50  0001 C CNN
 F 3 "~" H 9650 1150 50  0001 C CNN
 	1    9650 1150
@@
 $EndComp
 $Comp
-L Papilio_DUO-eagle-import:WE-CBF_0805 L?
+L Papilio_DUO-eagle-import:WE-CBF_0805 L100
 U 1 1 5BBBEFA0
 P 3650 2100
-F 0 "L?" H 3650 2100 59  0000 C CNN
+F 0 "L100" H 3650 2100 59  0000 C CNN
 F 1 "MH2029-300Y" H 3650 2000 59  0000 C CNN
-F 2 "" H 3650 2100 50  0001 C CNN
+F 2 "Papilio_DUO:0805" H 3650 2100 50  0001 C CNN
 F 3 "" H 3650 2100 50  0001 C CNN
 	1    3650 2100
@@
 AVCC
 $Comp
-L Papilio_DUO-eagle-import:C0603 C?
+L Papilio_DUO-eagle-import:C0603 C104
 U 1 1 5BBC6AF0
 P 4100 2200
-F 0 "C?" V 4060 2288 42  0000 L CNN
+F 0 "C104" V 4060 2288 42  0000 L CNN
 F 1 "1uF" V 4139 2288 42  0000 L CNN
-F 2 "" H 4100 2200 50  0001 C CNN
+F 2 "Papilio_DUO:0603" H 4100 2200 50  0001 C CNN
 F 3 "" H 4100 2200 50  0001 C CNN
 	1    4100 2200
@@
 Connection ~ 4100 2000
 $Comp
-L Papilio_DUO-eagle-import:C0603 C?
+L Papilio_DUO-eagle-import:C0603 C102
 U 1 1 5BBE6336
 P 4500 2300
-F 0 "C?" V 4460 2388 42  0000 L CNN
-F 1 "C0603" V 4539 2388 42  0000 L CNN
-F 2 "" H 4500 2300 50  0001 C CNN
+F 0 "C102" V 4460 2388 42  0000 L CNN
+F 1 "100nF" V 4539 2388 42  0000 L CNN
+F 2 "Papilio_DUO:0603" H 4500 2300 50  0001 C CNN
 F 3 "" H 4500 2300 50  0001 C CNN
 	1    4500 2300
@@
 $EndComp
 Wire Wire Line
-	4100 2000 5300 2000
+	4100 2000 4800 2000
 Connection ~ 5300 2000
 Wire Wire Line
@@
 	5050 2400 5250 2400
 $Comp
-L Papilio_DUO-eagle-import:ATMEGA32U4-XUMU U?
+L Papilio_DUO-eagle-import:ATMEGA32U4-XUMU U101
 U 1 1 5BB959E0
 P 6400 1900
-F 0 "U?" H 6600 3086 59  0000 C CNN
+F 0 "U101" H 6600 3086 59  0000 C CNN
 F 1 "ATMEGA32U4-XUMU" H 6600 2981 59  0000 C CNN
-F 2 "" H 6400 1900 50  0001 C CNN
+F 2 "Papilio_DUO:QFN44ML7X7" H 6400 1900 50  0001 C CNN
 F 3 "" H 6400 1900 50  0001 C CNN
 	1    6400 1900
@@
 UCAP
 $Comp
-L Papilio_DUO-eagle-import:C0603 C?
+L Papilio_DUO-eagle-import:C0603 C103
 U 1 1 5BC490EF
 P 4300 3000
-F 0 "C?" V 4260 3088 42  0000 L CNN
+F 0 "C103" V 4260 3088 42  0000 L CNN
 F 1 "1uF" V 4339 3088 42  0000 L CNN
-F 2 "" H 4300 3000 50  0001 C CNN
+F 2 "Papilio_DUO:0603" H 4300 3000 50  0001 C CNN
 F 3 "" H 4300 3000 50  0001 C CNN
 	1    4300 3000
@@
 $EndComp
 Wire Wire Line
-	4300 3100 5400 3100
+	4300 3100 4400 3100
 Wire Wire Line
 	7800 1000 8250 1000
@@
 	7800 2400 8250 2400
 $Comp
-L power:GND #PWR?
+L power:GND #PWR056
 U 1 1 5BC791C2
 P 8250 2400
-F 0 "#PWR?" H 8250 2150 50  0001 C CNN
+F 0 "#PWR056" H 8250 2150 50  0001 C CNN
 F 1 "GND" H 8400 2350 50  0000 C CNN
 F 2 "" H 8250 2400 50  0001 C CNN
@@
 	5250 4000 5250 4150
 $Comp
-L power:GND #PWR?
+L power:GND #PWR055
 U 1 1 5BD22211
 P 5250 4150
-F 0 "#PWR?" H 5250 3900 50  0001 C CNN
+F 0 "#PWR055" H 5250 3900 50  0001 C CNN
 F 1 "GND" H 5255 3977 50  0000 C CNN
 F 2 "" H 5250 4150 50  0001 C CNN
@@
 Text HLabel 10400 2450 2    50   BiDi ~ 0
 AREF
+NoConn ~ 8250 2300
+NoConn ~ 5200 5600
+NoConn ~ 8250 2600
+NoConn ~ 8250 2700
+NoConn ~ 8250 2900
+NoConn ~ 8250 3000
+NoConn ~ 8250 3100
+NoConn ~ 8250 3200
+NoConn ~ 7800 2800
+NoConn ~ 8250 3300
+$Comp
+L power:PWR_FLAG #FLG0105
+U 1 1 5C413B99
+P 4800 2000
+F 0 "#FLG0105" H 4800 2075 50  0001 C CNN
+F 1 "PWR_FLAG" H 4800 2174 50  0000 C CNN
+F 2 "" H 4800 2000 50  0001 C CNN
+F 3 "~" H 4800 2000 50  0001 C CNN
+	1    4800 2000
+	1    0    0    -1
+$EndComp
+Connection ~ 4800 2000
+Wire Wire Line
+	4800 2000 5300 2000
+NoConn ~ 8250 1000
+NoConn ~ 8250 1200
+NoConn ~ 8250 1300
+NoConn ~ 8250 1400
+NoConn ~ 8250 1500
+NoConn ~ 8250 1700
+$Comp
+L power:GND #PWR0113
+U 1 1 5C4452C3
+P 4400 3100
+F 0 "#PWR0113" H 4400 2850 50  0001 C CNN
+F 1 "GND" H 4405 2927 50  0000 C CNN
+F 2 "" H 4400 3100 50  0001 C CNN
+F 3 "" H 4400 3100 50  0001 C CNN
+	1    4400 3100
+	1    0    0    -1
+$EndComp
+Connection ~ 4400 3100
+Wire Wire Line
+	4400 3100 5400 3100
 $EndSCHEMATC

Commit message: Se actualizan en el esquematico recomendacion de Diego Brengi. Tambien se importa al PCB para verificar que no hayan habido cambios en las netlist.
Connections:
- wire segments 137 -> 128
Changed lines of the file:
@@
 Text Label 4850 1200 0    50   ~ 0
 ARD_RESET
-Text Label 9700 1350 0    50   ~ 0
+Text Label 9700 2200 0    50   ~ 0
 ARD_RESET
-Text HLabel 10400 1350 2    50   Input ~ 0
+Text HLabel 10400 2200 2    50   Input ~ 0
 ARD_RESET
 Wire Wire Line
@@
 L Papilio_DUO-eagle-import:R-NORMAL0603 R110
 U 1 1 5BBBA97E
-P 9650 1150
-F 0 "R110" V 9696 1087 50  0000 R CNN
-F 1 "10K" V 9605 1087 50  0000 R CNN
-F 2 "Papilio_DUO:0603" V 9580 1150 50  0001 C CNN
-F 3 "~" H 9650 1150 50  0001 C CNN
-	1    9650 1150
+P 9650 2000
+F 0 "R110" V 9696 1937 50  0000 R CNN
+F 1 "10K" V 9605 1937 50  0000 R CNN
+F 2 "Papilio_DUO:0603" V 9580 2000 50  0001 C CNN
+F 3 "~" H 9650 2000 50  0001 C CNN
+	1    9650 2000
 	0    -1   -1   0
 $EndComp
 Wire Wire Line
-	9650 950  9650 800
+	9650 1800 9650 1650
 $Comp
 L power:+3V3 #PWR0107
 U 1 1 5BBBED82
-P 9650 800
-F 0 "#PWR0107" H 9650 650 50  0001 C CNN
-F 1 "+3V3" H 9665 973 50  0000 C CNN
-F 2 "" H 9650 800 50  0001 C CNN
-F 3 "" H 9650 800 50  0001 C CNN
-	1    9650 800
+P 9650 1650
+F 0 "#PWR0107" H 9650 1500 50  0001 C CNN
+F 1 "+3V3" H 9665 1823 50  0000 C CNN
+F 2 "" H 9650 1650 50  0001 C CNN
+F 3 "" H 9650 1650 50  0001 C CNN
+	1    9650 1650
 	1    0    0    -1
 $EndComp
@@
 	7800 1000 8250 1000
 Wire Wire Line
-	7800 1100 8250 1100
-Wire Wire Line
 	7800 1200 8250 1200
 Wire Wire Line
@@
 Wire Wire Line
 	7800 1700 8250 1700
-Wire Wire Line
-	7800 2000 8250 2000
-Wire Wire Line
-	7800 2100 8250 2100
 Wire Wire Line
 	7800 2300 8250 2300
@@
 Wire Wire Line
 	7800 3300 8250 3300
-Wire Wire Line
-	7800 3500 8250 3500
-Wire Wire Line
-	7800 3600 8250 3600
-Wire Wire Line
-	7800 3700 8250 3700
-Wire Wire Line
-	7800 3800 8250 3800
-Wire Wire Line
-	7800 4100 8250 4100
-Wire Wire Line
-	7800 4200 8250 4200
 Text Label 7850 1000 0    50   ~ 0
 ATMEGA_IO9*
 Text Label 7850 1100 0    50   ~ 0
 MEGA_D14
-Wire Wire Line
-	9700 1450 10400 1450
-Text Label 9700 1450 0    50   ~ 0
-MEGA_D14
-Text HLabel 10400 1450 2    50   BiDi ~ 0
+Text HLabel 8950 1100 2    50   BiDi ~ 0
 MEGA_D14
 Text Label 7850 1200 0    50   ~ 0
@@
 MEGA_D15
 Wire Wire Line
-	9700 1550 10400 1550
-Wire Wire Line
-	9700 1650 10400 1650
-Text Label 9700 1550 0    50   ~ 0
+	9650 2200 10400 2200
+Text HLabel 8950 2000 2    50   BiDi ~ 0
 MEGA_D16
-Text Label 9700 1650 0    50   ~ 0
-MEGA_D15
-Wire Wire Line
-	9650 1350 10400 1350
-Text HLabel 10400 1550 2    50   BiDi ~ 0
-MEGA_D16
-Text HLabel 10400 1650 2    50   BiDi ~ 0
+Text HLabel 8950 2100 2    50   BiDi ~ 0
 MEGA_D15
 Text Label 7850 2300 0    50   ~ 0
@@
 Text Label 7850 4200 0    50   ~ 0
 ATMEGA_A0
-Text Label 9700 1750 0    50   ~ 0
+Text HLabel 8950 3500 2    50   BiDi ~ 0
 MEGA_D28/A5
-Text Label 9700 1850 0    50   ~ 0
+Text HLabel 8950 3600 2    50   BiDi ~ 0
 MEGA_D30/A4
-Text Label 9700 1950 0    50   ~ 0
+Text HLabel 8950 3700 2    50   BiDi ~ 0
 MEGA_D32/A3
-Text Label 9700 2050 0    50   ~ 0
+Text HLabel 8950 3800 2    50   BiDi ~ 0
 MEGA_D34/A2
-Text Label 9700 2150 0    50   ~ 0
+Text HLabel 8950 4100 2    50   BiDi ~ 0
 ATMEGA_A1
-Text Label 9700 2250 0    50   ~ 0
-ATMEGA_A0
-Wire Wire Line
-	9700 1750 10400 1750
-Wire Wire Line
-	9700 1850 10400 1850
-Wire Wire Line
-	9700 1950 10400 1950
-Wire Wire Line
-	9700 2050 10400 2050
-Wire Wire Line
-	9700 2150 10400 2150
-Wire Wire Line
-	9700 2250 10400 2250
-Text HLabel 10400 1750 2    50   BiDi ~ 0
-MEGA_D28/A5
-Text HLabel 10400 1850 2    50   BiDi ~ 0
-MEGA_D30/A4
-Text HLabel 10400 1950 2    50   BiDi ~ 0
-MEGA_D32/A3
-Text HLabel 10400 2050 2    50   BiDi ~ 0
-MEGA_D34/A2
-Text HLabel 10400 2150 2    50   BiDi ~ 0
-ATMEGA_A1
-Text HLabel 10400 2250 2    50   BiDi ~ 0
+Text HLabel 8950 4200 2    50   BiDi ~ 0
 ATMEGA_A0
 Text Label 4950 3200 0    50   ~ 0
@@
 Wire Wire Line
 	4400 3100 5400 3100
+Wire Wire Line
+	7800 4200 8950 4200
+Wire Wire Line
+	7800 4100 8950 4100
+Wire Wire Line
+	7800 3800 8950 3800
+Wire Wire Line
+	7800 3700 8950 3700
+Wire Wire Line
+	7800 3600 8950 3600
+Wire Wire Line
+	7800 3500 8950 3500
+Wire Wire Line
+	7800 2100 8950 2100
+Wire Wire Line
+	7800 2000 8950 2000
+Wire Wire Line
+	7800 1100 8950 1100
 $EndSCHEMATC
