File: PRACTICA_FINAL/PROJECTO_KICAD/FINAL/FPGA-PHERIPHERAL.sch (KiCad schematic (older format))
At the start: 4 parts

Commit message: Actualizado el esquematico se enumera igual que el pdf. Se asignan todas las huellas lo unico que falta es la huella de un Arduino superpuesto Se corre DRC de esquematico y tambien se pasa a .NET y se levanta en el Kicad PCB sin errores
Parts:
- FLASH1: renamed from U?; footprint (none) -> Papilio_DUO:SO08-EIAJ
- OSC1: renamed from OSC?; footprint (none) -> Papilio_DUO:OSC1
- SW1: renamed from SW?; footprint (none) -> Papilio_DUO:6P-2CH-2.54-9.1X3.5X3.2+2H
- U$1: renamed from J?; footprint (none) -> Papilio_DUO:JTAG
Connections:
- no-connect marks 0 -> 6
Changed lines of the file:
@@
 $EndDescr
 $Comp
-L Papilio_DUO-eagle-import:JTAG_XILINX J?
+L Papilio_DUO-eagle-import:JTAG_XILINX U$1
 U 1 1 5BC3038B
 P 2350 2750
-F 0 "J?" H 2050 3200 59  0000 C CNN
+F 0 "U$1" H 2050 3200 59  0000 C CNN
 F 1 "JTAG_XILINX" H 2250 2400 59  0000 C CNN
-F 2 "" H 2350 2750 50  0001 C CNN
+F 2 "Papilio_DUO:JTAG" H 2350 2750 50  0001 C CNN
 F 3 "" H 2350 2750 50  0001 C CNN
 	1    2350 2750
@@
 AD3-JTAG_TMS
 $Comp
-L Papilio_DUO-eagle-import:OSC1 OSC?
+L Papilio_DUO-eagle-import:OSC1 OSC1
 U 1 1 5BC306FE
 P 2350 1550
-F 0 "OSC?" H 2350 1850 78  0000 C CNB
+F 0 "OSC1" H 2350 1850 78  0000 C CNB
 F 1 "32MHz" H 2350 1250 78  0000 C CNB
-F 2 "" H 2350 1550 50  0001 C CNN
+F 2 "Papilio_DUO:OSC1" H 2350 1550 50  0001 C CNN
 F 3 "" H 2350 1550 50  0001 C CNN
 	1    2350 1550
@@
 	1800 1450 1800 1300
 $Comp
-L power:+3V3 #PWR?
+L power:+3V3 #PWR020
 U 1 1 5BC309F1
 P 1800 1300
-F 0 "#PWR?" H 1800 1150 50  0001 C CNN
+F 0 "#PWR020" H 1800 1150 50  0001 C CNN
 F 1 "+3V3" H 1815 1473 50  0000 C CNN
 F 2 "" H 1800 1300 50  0001 C CNN
@@
 	2850 1650 2850 1750
 $Comp
-L power:GND #PWR?
+L power:GND #PWR021
 U 1 1 5BC31188
 P 2850 1750
-F 0 "#PWR?" H 2850 1500 50  0001 C CNN
+F 0 "#PWR021" H 2850 1500 50  0001 C CNN
 F 1 "GND" H 2855 1577 50  0000 C CNN
 F 2 "" H 2850 1750 50  0001 C CNN
@@
 $EndComp
 $Comp
-L Papilio_DUO-eagle-import:FLASH-SPI-25XXSMD1 U?
+L Papilio_DUO-eagle-import:FLASH-SPI-25XXSMD1 FLASH1
 U 1 1 5BC31998
 P 2450 4000
-F 0 "U?" H 2450 4347 42  0000 C CNN
+F 0 "FLASH1" H 2450 4347 42  0000 C CNN
 F 1 "FLASH-SPI-25XXSMD1" H 2450 4268 42  0000 C CNN
-F 2 "" H 2450 4000 50  0001 C CNN
+F 2 "Papilio_DUO:SO08-EIAJ" H 2450 4000 50  0001 C CNN
 F 3 "" H 2450 4000 50  0001 C CNN
 	1    2450 4000
@@
 	1050 4100 1050 4050
 $Comp
-L power:+3V3 #PWR?
+L power:+3V3 #PWR018
 U 1 1 5BC321A7
 P 1050 4050
-F 0 "#PWR?" H 1050 3900 50  0001 C CNN
+F 0 "#PWR018" H 1050 3900 50  0001 C CNN
 F 1 "+3V3" H 1065 4223 50  0000 C CNN
 F 2 "" H 1050 4050 50  0001 C CNN
@@
 	1050 4200 1050 4250
 $Comp
-L power:GND #PWR?
+L power:GND #PWR019
 U 1 1 5BC324F1
 P 1050 4250
-F 0 "#PWR?" H 1050 4000 50  0001 C CNN
+F 0 "#PWR019" H 1050 4000 50  0001 C CNN
 F 1 "GND" H 1055 4077 50  0000 C CNN
 F 2 "" H 1050 4250 50  0001 C CNN
@@
 	3200 3900 3200 3800
 $Comp
-L power:+3V3 #PWR?
+L power:+3V3 #PWR024
 U 1 1 5BC3406C
 P 3200 3800
-F 0 "#PWR?" H 3200 3650 50  0001 C CNN
+F 0 "#PWR024" H 3200 3650 50  0001 C CNN
 F 1 "+3V3" H 3215 3973 50  0000 C CNN
 F 2 "" H 3200 3800 50  0001 C CNN
@@
 	7600 1600 8250 1600
 $Comp
-L Papilio_DUO-eagle-import:SWITCH-2CH-6P-3010010P1 SW?
+L Papilio_DUO-eagle-import:SWITCH-2CH-6P-3010010P1 SW1
 U 1 1 5BC3AB52
 P 2450 5050
-F 0 "SW?" H 2450 5357 42  0000 C CNN
+F 0 "SW1" H 2450 5357 42  0000 C CNN
 F 1 "SWITCH-2CH-6P-3010010P1" H 2450 5278 42  0000 C CNN
-F 2 "" H 2450 5050 50  0001 C CNN
+F 2 "Papilio_DUO:6P-2CH-2.54-9.1X3.5X3.2+2H" H 2450 5050 50  0001 C CNN
 F 3 "" H 2450 5050 50  0001 C CNN
 	1    2450 5050
@@
 	3050 4950 3050 4700
 $Comp
-L power:+3V3 #PWR?
+L power:+3V3 #PWR022
 U 1 1 5BC3D41C
 P 3050 4700
-F 0 "#PWR?" H 3050 4550 50  0001 C CNN
+F 0 "#PWR022" H 3050 4550 50  0001 C CNN
 F 1 "+3V3" H 3065 4873 50  0000 C CNN
 F 2 "" H 3050 4700 50  0001 C CNN
@@
 	3050 5150 3050 5300
 $Comp
-L power:GND #PWR?
+L power:GND #PWR023
 U 1 1 5BC3DB65
 P 3050 5300
-F 0 "#PWR?" H 3050 5050 50  0001 C CNN
+F 0 "#PWR023" H 3050 5050 50  0001 C CNN
 F 1 "GND" H 3055 5127 50  0000 C CNN
 F 2 "" H 3050 5300 50  0001 C CNN
@@
 Text HLabel 8250 2850 2    50   BiDi ~ 0
 SW1
+NoConn ~ 2100 4950
+NoConn ~ 2100 5050
+NoConn ~ 2100 5150
+NoConn ~ 2900 2450
+NoConn ~ 2900 2550
+NoConn ~ 3300 2400
 $EndSCHEMATC

Commit message: Se conecta la señal de JTAG_REG del conector JTAG estaba conectado en el PCB y en el esquematico no se vio conectado. Se hace la modificacion en el esquematico y se hace backannotate al PCB:
Connections:
- wire segments 40 -> 41
Changed lines of the file:
@@
 $EndComp
-Wire Wire Line
-	2650 2450 2900 2450
 Wire Wire Line
 	2650 2550 2900 2550
@@
 NoConn ~ 2900 2550
 NoConn ~ 3300 2400
+Wire Wire Line
+	3200 2450 3200 2250
+Wire Wire Line
+	2650 2450 3200 2450
+$Comp
+L power:+3V3 #PWR?
+U 1 1 5BCC6E17
+P 3200 2250
+F 0 "#PWR?" H 3200 2100 50  0001 C CNN
+F 1 "+3V3" H 3215 2423 50  0000 C CNN
+F 2 "" H 3200 2250 50  0001 C CNN
+F 3 "" H 3200 2250 50  0001 C CNN
+	1    3200 2250
+	1    0    0    -1
+$EndComp
 $EndSCHEMATC

Commit message: Se actualizan en el esquematico recomendacion de Diego Brengi. Tambien se importa al PCB para verificar que no hayan habido cambios en las netlist.
Connections:
- wire segments 41 -> 35
