File: PRACTICA_FINAL/PROJECTO_KICAD/FINAL/FT2232H.sch (KiCad schematic (older format))
At the start: 31 parts

Commit message: Actualizado el esquematico se enumera igual que el pdf. Se asignan todas las huellas lo unico que falta es la huella de un Arduino superpuesto Se corre DRC de esquematico y tambien se pasa a .NET y se levanta en el Kicad PCB sin errores
Parts:
- C14, C19, C28: renamed from C?; footprint (none) -> Papilio_DUO:SMC_A
- C15, C16, C17, C18, C20, C27, C29, C30, C31, C34, C8, C9: renamed from C?; footprint (none) -> Papilio_DUO:0603
- FPGAUSB1: renamed from CONN?; footprint (none) -> Papilio_DUO:CONN_USB_MINI-B
- IC1: renamed from U?; footprint (none) -> Papilio_DUO:LQFP64
- L3, L4: renamed from L?; footprint (none) -> Papilio_DUO:FB603
- R23, R24, R25, R26, R27, R28, R29, R30: renamed from R?; footprint (none) -> Papilio_DUO:0603
- RX1: renamed from D?; value RX -> LEDCHIP-LED0805; footprint (none) -> Papilio_DUO:CHIP-LED0805; symbol Device:LED -> Papilio_DUO-eagle-import:LEDCHIP-LED0805
- TX1: renamed from D?; value TX -> LEDCHIP-LED0805; footprint (none) -> Papilio_DUO:CHIP-LED0805; symbol Device:LED -> Papilio_DUO-eagle-import:LEDCHIP-LED0805
- U3: renamed from U?; footprint (none) -> Papilio_DUO:SOT23-6
- X1: renamed from X?; footprint (none) -> Papilio_DUO:4X6
Connections:
- net labels removed: 3.3V
- wire segments 143 -> 149
- no-connect marks 0 -> 23

Commit message: Se actualizan en el esquematico recomendacion de Diego Brengi. Tambien se importa al PCB para verificar que no hayan habido cambios en las netlist.
Connections:
- wire segments 149 -> 151
Changed lines of the file:
@@
 $EndComp
 Wire Wire Line
-	3150 1100 5100 1100
+	3150 1100 4450 1100
 Wire Wire Line
 	5100 1100 5100 1850
@@
 Connection ~ 4150 1400
 Wire Wire Line
-	4150 1400 4600 1400
+	4150 1400 4450 1400
 Wire Wire Line
 	3700 1450 3700 1400
@@
 NoConn ~ 7800 5850
 NoConn ~ 1150 2700
-$Comp
-L power:PWR_FLAG #FLG0106
-U 1 1 5C44563D
-P 5600 1200
-F 0 "#FLG0106" H 5600 1275 50  0001 C CNN
-F 1 "PWR_FLAG" H 5600 1374 50  0000 C CNN
-F 2 "" H 5600 1200 50  0001 C CNN
-F 3 "~" H 5600 1200 50  0001 C CNN
-	1    5600 1200
-	1    0    0    -1
-$EndComp
 Wire Wire Line
 	5600 1200 5600 1750
@@
 Wire Wire Line
 	10400 4750 10400 4800
+$Comp
+L power:PWR_FLAG #FLG0107
+U 1 1 5BF0EF4A
+P 4450 1100
+F 0 "#FLG0107" H 4450 1175 50  0001 C CNN
+F 1 "PWR_FLAG" H 4450 1274 50  0000 C CNN
+F 2 "" H 4450 1100 50  0001 C CNN
+F 3 "~" H 4450 1100 50  0001 C CNN
+	1    4450 1100
+	1    0    0    -1
+$EndComp
+Connection ~ 4450 1100
+Wire Wire Line
+	4450 1100 5100 1100
+$Comp
+L power:PWR_FLAG #FLG0108
+U 1 1 5BF0EF95
+P 4450 1400
+F 0 "#FLG0108" H 4450 1475 50  0001 C CNN
+F 1 "PWR_FLAG" H 4450 1574 50  0000 C CNN
+F 2 "" H 4450 1400 50  0001 C CNN
+F 3 "~" H 4450 1400 50  0001 C CNN
+	1    4450 1400
+	1    0    0    -1
+$EndComp
+Connection ~ 4450 1400
+Wire Wire Line
+	4450 1400 4600 1400
 $EndSCHEMATC
